File: fat_cruiser/v1/main.kicad_pcb (KiCad board)
At the start: 2 copper layers, 222.2 x 100.1 mm, 92 parts

Commit message: Work on pcb
Parts:
- moved D19 19.3 mm to (261.7, 95.1), turned to 10 degrees
- moved S19 19.0 mm to (260.8, 90.1), turned to 10 degrees
- moved D20 18.4 mm to (258.7, 78.3), turned to 10 degrees
- moved S20 18.2 mm to (257.9, 73.4), turned to 10 degrees
- moved D21 17.9 mm to (255.8, 61.6), turned to 10 degrees
- moved S21 17.8 mm to (254.9, 56.7), turned to 10 degrees
- moved _4 17.8 mm to (254.9, 82.5), turned to 10 degrees
- moved D1 17.8 mm to (54.5, 95.1), turned to -10 degrees
- moved S1 17.4 mm to (55.4, 90.1), turned to -10 degrees
- moved D2 16.8 mm to (57.5, 78.3), turned to -10 degrees
- moved ? 16.7 mm to (244.4, 100.8), turned to 10 degrees
- moved S2 16.6 mm to (58.4, 73.4), turned to -10 degrees
- moved D3 16.3 mm to (60.4, 61.6), turned to -10 degrees
- moved S3 16.3 mm to (61.3, 56.7), turned to -10 degrees
- moved _3 16.2 mm to (61.3, 82.5), turned to -10 degrees
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Routing:
- net P26: track 183.6 -> 233.8 mm
- net P27: track 168.0 -> 168.8 mm
Other:
- board size 222.2 x 100.1 mm -> 225.6 x 86.5 mm

Commit message: Add gerber files
Parts:
- moved _18 8.32 mm to (158.8, 103.2)
- moved D16 8.32 mm to (91.9, 97.9)
- moved D14 8.32 mm to (128.8, 69.9)
- moved S31 8.32 mm to (185.8, 81.7)
- moved D21 8.32 mm to (254.0, 53.5)
- moved S36 8.32 mm to (184.4, 99.2)
- moved _16 8.32 mm to (153.8, 103.2)
- moved S4 8.32 mm to (74.1, 69.4)
- moved D5 8.32 mm to (76.2, 57.6)
- moved S18 8.32 mm to (128.2, 99.2)
- moved S24 8.32 mm to (232.6, 35.9)
- moved S33 8.32 mm to (179.9, 48.2)
- moved S6 8.32 mm to (80.0, 35.9)
- moved _13 8.32 mm to (109.9, 47.8)
- moved _15 8.32 mm to (151.2, 103.2)
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Routing:
- net GND: track 375.6 -> 632.7 mm
- net P22: track 108.8 -> 159.7 mm
- net P10: track 197.4 -> 193.2 mm
- net P5: track 368.5 -> 372.1 mm
- net P9: track 332.4 -> 331.1 mm
- net P3: track 329.6 -> 330.6 mm
- net P6: track 198.5 -> 197.6 mm
- net P27: track 168.8 -> 168.0 mm
