File: fat_cruiser/v2/main.kicad_pcb (KiCad board)
At the start: 2 copper layers, 225.6 x 86.5 mm, 92 parts

Commit message: Work on v2
Parts:
- removed ? (x2): , text
- removed _10, _11, _12, _13, _14, _15, _16, _17, _18, _19, _6, _7, _8, _9: , MountingHole_Pad_Via
- added MH1: , MountingHole_Pad_Via, F.Cu at (57.4, 115.8)
- added MH10: , MountingHole_Pad_Via, F.Cu at (246.2, 65.6)
- added MH2: , MountingHole_Pad_Via, F.Cu at (247.6, 115.8)
- added MH3: , MountingHole_Pad_Via, F.Cu at (135.2, 117.5)
- added MH4: , MountingHole_Pad_Via, F.Cu at (169.8, 117.5)
- added MH5: , MountingHole_Pad_Via, F.Cu at (137.9, 83.3)
- added MH6: , MountingHole_Pad_Via, F.Cu at (167.1, 83.3)
- added MH7: , MountingHole_Pad_Via, F.Cu at (138.9, 155.1)
- added MH8: , MountingHole_Pad_Via, F.Cu at (166.1, 155.1)
- added MH9: , MountingHole_Pad_Via, F.Cu at (58.8, 65.6)
- added OLED1: , OLED_SSD1306, F.Cu at (152.5, 123.2)
- added T1: , text, F.Cu at (60.8, 121.5)
- added T2: , text, F.Cu at (244.3, 121.5)
- added _1: , MountingHole_Pad_Via, F.Cu at (147.4, 155.6)
- added _2: , MountingHole_Pad_Via, F.Cu at (150.0, 155.6)
- moved _4 127.3 mm to (155.0, 155.6), turned to 0 degrees
- moved _3 123.5 mm to (152.5, 155.6), turned to 0 degrees
- moved _5 73.1 mm to (157.6, 155.6), turned to 0 degrees
- moved S18 52.8 mm to (122.0, 151.6), turned to -55 degrees
- moved S36 52.4 mm to (183.1, 151.6), turned to 55 degrees
- moved D18 51.2 mm to (117.9, 154.5), turned to -55 degrees
- moved D36 50.4 mm to (187.2, 154.5), turned to 55 degrees
- moved S35 41.1 mm to (196.4, 136.8), turned to 41 degrees
- moved S17 40.7 mm to (108.6, 136.8), turned to -41 degrees
- moved D17 39.8 mm to (105.3, 140.6), turned to -41 degrees
- moved D35 39.7 mm to (199.7, 140.6), turned to 41 degrees
- moved D10 35.6 mm to (99.4, 112.9), turned to -12 degrees
- moved S10 35.6 mm to (100.4, 108.0), turned to -12 degrees
- moved D11 35.6 mm to (102.9, 96.3), turned to -12 degrees
- moved S11 35.6 mm to (104.0, 91.4), turned to -12 degrees
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Routing:
- net GND: track 632.7 -> 541.6 mm
- net P26: track 233.8 -> 149.1 mm
- net P5: track 372.1 -> 293.1 mm
- net P2: track 75.1 -> 128.6 mm
- net P8: track 209.6 -> 159.0 mm
- net 3V3_OUT: track 0.00 -> 44.7 mm
- net P3: track 330.6 -> 288.1 mm
- net P6: track 197.6 -> 155.3 mm
- net P10: track 193.2 -> 231.4 mm
- net P27: track 168.0 -> 138.7 mm
- net P21: track 90.1 -> 119.3 mm
- net P7: track 165.5 -> 136.4 mm
- net P22: track 159.7 -> 131.3 mm
- net P9: track 331.1 -> 305.1 mm
- net P28: track 186.7 -> 161.9 mm
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Other:
- board size 225.6 x 86.5 mm -> 239.7 x 107.3 mm
